Commit message: added initial joint configuration so that inverse kinematics converges

File: code/marker.urdf (robot description, URDF)
Before this commit: robot milling_head, 2 links, 1 joints
Joints:
- joint milling_trafo: origin xyz=0.0 0.0 0.0 rpy=0 0 0 -> xyz=0.0 0.0 0.0 rpy=0 -1.57075 0

Commit message: adjusted experiment to new interface

File: code/marker.urdf (robot description, URDF)
Before this commit: robot milling_head, 2 links, 1 joints
Joints:
- joint milling_trafo: origin xyz=0.0 0.0 0.0 rpy=0 -1.57075 0 -> xyz=0.0 0.0 0.0 rpy=0 0 0
