Commit message: added distance to obective and fixed module collision shape

File: code/transformer_cell/Objects/modules/milling_module.urdf (robot description, URDF)
Before this commit: robot milling_module, 1 links, 0 joints
Links:
- link baseLink: geometry collision mesh filename=mesh/Fraesmodul_dec.stl; visual mesh filename=mesh/Fraesmodul_dec.stl

Commit message: fixed bug in distance constraint where 1.2 was evaluated after sum

File: code/transformer_cell/Objects/modules/milling_module.urdf (robot description, URDF)
Before this commit: robot milling_module, 1 links, 0 joints
Links:
- link baseLink: geometry collision box size=1200 1200 1000; visual mesh filename=mesh/Fraesmodul_dec.stl

Commit message: added concave mesh to experiment

File: code/transformer_cell/Objects/modules/milling_module.urdf (robot description, URDF)
Before this commit: robot milling_module, 1 links, 0 joints
Links:
- link baseLink: mass 1 -> None; geometry collision mesh filename=mesh/Fraesmodul_dec.stl; visual mesh filename=mesh/Fraesmodul_dec.stl
